File: tangnano9k_brushless_driver.kicad_pcb (KiCad board)
At the start: 2 copper layers, 99.9 x 99.9 mm, 6 parts, among them J1 Nucleo_F302R8, J2 Conn_01x08_Socket, U1 Tang_Nano_9k_board, U2 MCP3008

Commit message: 0906
Parts:
- moved U2 72.2 mm to (142.5, 77.5)
- moved C1 70.4 mm to (150.2, 73.7)
- moved PS1 63.7 mm to (139.7, 112.3), turned to 90 degrees
- moved J2 11.5 mm to (155.4, 145.3)
- moved U1 10.3 mm to (171.5, 118.6)
- moved J1 8.46 mm to (129.5, 86.9)
Connections:
- U1 pad 12: unconnected-(U1-34/IOB23B/RGB_VS-Pad12) -> /H_V
- U1 pad 13: unconnected-(U1-40/IOB33B/RGB_HS-Pad13) -> /H_W
- U1 pad 17: /_LIN_S -> unconnected-(U1-51/IOR17B/RGB_B5-Pad17)
- U1 pad 18: /HIN_T -> unconnected-(U1-53/IOR15B/RGB_B4-Pad18)
- U1 pad 19: /_LIN_R -> unconnected-(U1-54/IOR15A/RGB_B3-Pad19)
- U1 pad 20: /_LIN_T -> unconnected-(U1-55/IOR14B/RGB_G7-Pad20)
- U1 pad 21: /DIRECTION -> unconnected-(U1-56/IOR14A/RGB_G6-Pad21)
- U1 pad 22: /D_IN -> unconnected-(U1-57/IOR13A/RGB_G5-Pad22)
- U1 pad 23: /HIN_S -> /D_IN
- U1 pad 24: /HIN_R -> /DIRECTION
- U1 pad 8: /H_W -> unconnected-(U1-28/IOB11B-Pad8)
- U1 pad 9: /H_V -> unconnected-(U1-29/IOB13A-Pad9)
Routing:
- net /5V: track 0.00 -> 29.0 mm
- net +3.3V: track 0.00 -> 24.9 mm
- net Net-(U1-31/IOB15A/RGB_TOUCH_YD): track 0.00 -> 17.7 mm
- net Net-(U1-32/IOB15B/RGB_TOUCH_XR): track 0.00 -> 17.7 mm
- net /H_V: track 0.00 -> 10.9 mm
- net /VIN12: track 0.00 -> 9.56 mm
- net /H_W: track 0.00 -> 7.62 mm
- net /D_IN: track 0.00 -> 7.62 mm
- net /DIRECTION: track 0.00 -> 7.62 mm

Commit message: 0907
Parts:
- added JP1: SolderJumper_2_Open, Jumper:SolderJumper-2_P1.3mm_Open_TrianglePad1.0x1.5mm, F.Cu at (153.4, 81.3)
- added R1: R, Resistor_SMD:R_0603_1608Metric_Pad0.98x0.95mm_HandSolder, F.Cu at (157.0, 81.3)
- added R2: R, Resistor_SMD:R_0603_1608Metric_Pad0.98x0.95mm_HandSolder, F.Cu at (157.0, 84.6)
- C1: footprint Capacitor_THT:C_Axial_L3.8mm_D2.6mm_P7.50mm_Horizontal -> Capacitor_SMD:C_0603_1608Metric_Pad1.08x0.95mm_HandSolder
- moved C1 10.3 mm to (151.9, 83.8), turned to -90 degrees
- moved U2 2.54 mm to (142.2, 80.0)
Connections:
- C1 pad 1: +3.3V -> Net-(JP1-A)
- U1 pad 10: /H_U -> unconnected-(U1-30/IOB13B-Pad10)
- U1 pad 11: unconnected-(U1-33/IOB23A/RGB_DE-Pad11) -> /H_U
- U2 pad 1: /C7-28 -> /C10-11
- U2 pad 15: +3.3V -> Net-(JP1-A)
- U2 pad 2: /C7-36 -> /C10-28
- U2 pad 3: /C7-38 -> /C10-34
- U2 pad 4: /C10-28 -> /C7-38
- U2 pad 5: /C10-34 -> /ACCEL
- U2 pad 6: /A_IN -> /C7-36
- U2 pad 7: /ACCEL -> /A_IN
- U2 pad 8: /C10-11 -> /C7-28
Routing:
- net /C10-34: track 0.00 -> 127.4 mm
- net /H_U: track 0.00 -> 114.9 mm
- net /C10-28: track 0.00 -> 111.2 mm
- net /C7-38: track 0.00 -> 84.7 mm
- net /C10-11: track 0.00 -> 82.1 mm
- net /C7-36: track 0.00 -> 80.4 mm
- net /ACCEL: track 0.00 -> 79.9 mm
- net /A_IN: track 0.00 -> 74.7 mm
- net /C7-28: track 0.00 -> 68.3 mm
- net Net-(U1-41/IOB41A/RGB_B7): track 0.00 -> 40.1 mm
- net Net-(U1-42IOB41B/RGB_B6): track 0.00 -> 40.1 mm
- net +3.3V: track 24.9 -> 57.1 mm
- net Net-(JP1-A): track 0.00 -> 9.19 mm
- net Net-(U1-31/IOB15A/RGB_TOUCH_YD): track 17.7 -> 13.0 mm
- net Net-(U1-32/IOB15B/RGB_TOUCH_XR): track 17.7 -> 13.0 mm
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Other:
- board text added: "#LIN_R"
- board text added: "#LIN_S"
- board text added: "#LIN_T"
- board text added: "1"
- board text added: "12V"
- board text added: "2"
- board text added: "25"
- board text added: "26"
- board text added: "27"
- board text added: "28"
- board text added: "29"
- board text added: "30"
- board text added: "31/Dout"
- board text added: "32/CLK"
- board text added: "33/H_U"
- board text added: "34/H_V"
- board text added: "35"
- board text added: "37"
- board text added: "38"
- board text added: "3V3"
- board text added: "40/H_W"
- board text added: "41/CS SHDN"
- board text added: "42/Din"
- board text added: "48"
- board text added: "49"
- board text added: "56"
- board text added: "57"
- board text added: "5V"
- board text added: "63"
- board text added: "68/D_IN"
- board text added: "69/DIRECTION"
- board text added: "70"
- board text added: "74"
- board text added: "77"
- board text added: "79"
- board text added: "86"
- board text added: "<HDMI>"
- board text added: "<USB>"
- board text added: "A1"
- board text added: "A8"
- board text added: "ACCEL"
- board text added: "AGND"
- board text added: "A_IN"
- board text added: "CLK"
- board text added: "CN2"
- board text added: "CS/SHDN"
- board text added: "DGND"
- board text added: "DIR"
- board text added: "Din"
- board text added: "Dout"
- board text added: "GND"
- board text added: "HIN_R"
- board text added: "HIN_S"
- board text added: "HIN_T"
- board text added: "H_U"
- board text added: "H_V"
- board text added: "H_W"
- board text added: "I/O 1.8V"
- board text added: "Ref"

Commit message: 0908
Parts:
- added J3: Conn_01x04_Socket, Connector_PinSocket_2.54mm:PinSocket_1x04_P2.54mm_Vertical, F.Cu at (187.8, 147.8)
- added R10: R, Resistor_SMD:R_0603_1608Metric_Pad0.98x0.95mm_HandSolder, B.Cu at (187.3, 66.5)
- added R3: R, Resistor_SMD:R_0603_1608Metric_Pad0.98x0.95mm_HandSolder, B.Cu at (155.8, 66.5)
- added R4: R, Resistor_SMD:R_0603_1608Metric_Pad0.98x0.95mm_HandSolder, B.Cu at (159.3, 66.5)
- added R5: R, Resistor_SMD:R_0603_1608Metric_Pad0.98x0.95mm_HandSolder, B.Cu at (162.8, 66.5)
- added R6: R, Resistor_SMD:R_0603_1608Metric_Pad0.98x0.95mm_HandSolder, B.Cu at (166.2, 66.5)
- added R7: R, Resistor_SMD:R_0603_1608Metric_Pad0.98x0.95mm_HandSolder, B.Cu at (169.8, 66.5)
- added R8: R, Resistor_SMD:R_0603_1608Metric_Pad0.98x0.95mm_HandSolder, B.Cu at (176.8, 66.5)
- added R9: R, Resistor_SMD:R_0603_1608Metric_Pad0.98x0.95mm_HandSolder, B.Cu at (190.8, 66.5)
- added S1: TVGP01-G73BB, samacsys:TVGP01G73BB, F.Cu at (138.3, 143.2)
- added S2: TVGP01-G73BB, samacsys:TVGP01G73BB, F.Cu at (134.3, 148.2)
- added S3: TVGP01-G73BB, samacsys:TVGP01G73BB, F.Cu at (138.2, 129.2)
- added S4: TVGP01-G73BB, samacsys:TVGP01G73BB, F.Cu at (143.6, 115.0)
- added SW1: SW_SPDT, Connector_PinHeader_2.54mm:PinHeader_1x03_P2.54mm_Vertical, F.Cu at (134.1, 60.8)
- added SW2: SW_SPDT, Connector_PinHeader_2.54mm:PinHeader_1x03_P2.54mm_Vertical, F.Cu at (124.1, 60.8)
- added U3: C-574SR-LF, Library:C-574SR-LF, F.Cu at (155.8, 59.9)
- C1: footprint Capacitor_SMD:C_0603_1608Metric_Pad1.08x0.95mm_HandSolder -> Connector:FanPinHeader_1x03_P2.54mm_Vertical
Connections:
- net +3.3V renamed +3V3
- U1 pad 1: unconnected-(U1-38/IOB31B/TF_CS-Pad1) -> Net-(J3-Pin_1)
- U1 pad 10: unconnected-(U1-30/IOB13B-Pad10) -> /DIG1
- U1 pad 11: /H_U -> Net-(U1-33/IOB23A/RGB_DE)
- U1 pad 12: /H_V -> /DIG3
- U1 pad 13: /H_W -> /DIG2
- U1 pad 14: unconnected-(U1-35/IOB29A/RGB_CK-Pad14) -> Net-(U1-35/IOB29A/RGB_CK)
- U1 pad 15: Net-(U1-41/IOB41A/RGB_B7) -> /H_V
- U1 pad 16: Net-(U1-42IOB41B/RGB_B6) -> /H_W
- U1 pad 2: unconnected-(U1-37/IO31A/TF_MOSI-Pad2) -> Net-(J3-Pin_2)
- U1 pad 21: unconnected-(U1-56/IOR14A/RGB_G6-Pad21) -> /Anode_A
- U1 pad 22: unconnected-(U1-57/IOR13A/RGB_G5-Pad22) -> /DIG4
- U1 pad 29: unconnected-(U1-49/IOR24A/SPILCD_RS-Pad29) -> /Din
- U1 pad 3: unconnected-(U1-36/IOB29B/TF_SCK-Pad3) -> Net-(J3-Pin_3)
- U1 pad 30: unconnected-(U1-48/IOR24B/SPILCD_CS-Pad30) -> /CS/SHDN
- U1 pad 32: unconnected-(U1-70/IOT41B/RGB_G2/HDMI_C0N-Pad32) -> Net-(S4-NO_1)
- U1 pad 33: unconnected-(U1-71/IOT41A/RGB_R7/HDMI_D0P-Pad33) -> Net-(S3-NO_1)
- U1 pad 34: unconnected-(U1-72/IOT39B/RGB_R6/HDMI_D1N-Pad34) -> Net-(S2-NO_1)
- U1 pad 35: unconnected-(U1-73/IOT39A/RGB_R5/HDMI_D1P-Pad35) -> Net-(S1-NO_1)
- U1 pad 38: unconnected-(U1-76/IOT37B/SPILCD_CK-Pad38) -> Net-(SW2-B)
- U1 pad 39: unconnected-(U1-77/IOT37A/SPILCD_MO-Pad39) -> Net-(SW1-B)
- U1 pad 4: unconnected-(U1-39/IOB33A/TF_MISO-Pad4) -> Net-(J3-Pin_4)
- U1 pad 48: unconnected-(U1-63/IOR5A/RGB_TOUCH_XL-Pad48) -> /H_U
- U1 pad 5: unconnected-(U1-25/IOB8A-Pad5) -> Net-(U1-25/IOB8A)
- U1 pad 6: unconnected-(U1-26/IOB8B-Pad6) -> Net-(U1-26/IOB8B)
- U1 pad 7: unconnected-(U1-27/IOB11A-Pad7) -> Net-(U1-27/IOB11A)
- U1 pad 8: unconnected-(U1-28/IOB11B-Pad8) -> Net-(U1-28/IOB11B)
- U1 pad 9: unconnected-(U1-29/IOB13A-Pad9) -> Net-(U1-29/IOB13A)
- U2 pad 10: Net-(U1-41/IOB41A/RGB_B7) -> /CS/SHDN
- U2 pad 11: Net-(U1-42IOB41B/RGB_B6) -> /Din
Routing:
- net +3V3: track 57.1 -> 166.9 mm
- net Net-(SW2-B): track 0.00 -> 91.8 mm
- net Net-(SW1-B): track 0.00 -> 87.0 mm
- net Net-(U1-25/IOB8A): track 0.00 -> 85.6 mm
- net Net-(U1-26/IOB8B): track 0.00 -> 81.6 mm
- net Net-(U1-27/IOB11A): track 0.00 -> 77.8 mm
- net Net-(U1-28/IOB11B): track 0.00 -> 74.1 mm
- net /DIG1: track 0.00 -> 73.7 mm
- net Net-(U1-29/IOB13A): track 0.00 -> 70.4 mm
- net /DIG3: track 0.00 -> 68.6 mm
- net /DIG2: track 0.00 -> 65.9 mm
- net Net-(U1-33/IOB23A/RGB_DE): track 0.00 -> 63.7 mm
- net Net-(U1-35/IOB29A/RGB_CK): track 0.00 -> 55.7 mm
- net Net-(S1-NO_1): track 0.00 -> 46.2 mm
- net Net-(S2-NO_1): track 0.00 -> 45.7 mm
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- added copper zone on B.Cu, net GND
- added copper zone on F.Cu, net GND
Other:
- board size 99.9 x 99.9 mm -> 81.5 x 99.9 mm
- board text added: "33"
- board text added: "34"
- board text added: "36"
- board text added: "39"
- board text added: "40"
- board text added: "41/H_V"
- board text added: "42/H_W"
- board text added: "48/CS SHDN"
- board text added: "49/Din"
- board text added: "51"
- board text added: "53"
- board text added: "54"
- board text added: "55"
- board text added: "63/H_U"
- board text added: "71"
- board text added: "72"
- board text added: "73"
- board text added: "75"
- board text added: "76"
- board text added: "A"
- board text added: "B"
- board text added: "C"
- board text added: "D"
- board text added: "DIG1"
- board text added: "DIG2"
- board text added: "DIG3"
- board text added: "DIG4"
- board text added: "DP"
- board text added: "E"
- board text added: "F"
- board text added: "G"
- board text added: "[BP5293-50]"
- board text added: "[C-574SR-LF]"
- board text added: "[MCP3008]"
- board text added: "[Tang Nano 9K]"
- board text removed: "33/H_U"
- board text removed: "34/H_V"
- board text removed: "40/H_W"
- board text removed: "41/CS SHDN"
- board text removed: "42/Din"
- board text removed: "48"
- board text removed: "49"
- board text removed: "63"

Commit message: 0909
Parts:
- added G***: LOGO, MyLibrary:kamo20, F.Cu at (129.0, 74.7)
- added SW3: SW_SPDT, Connector_PinHeader_2.54mm:PinHeader_1x03_P2.54mm_Vertical, F.Cu at (124.0, 60.7)
- C1: footprint Connector:FanPinHeader_1x03_P2.54mm_Vertical -> Capacitor_SMD:C_0603_1608Metric_Pad1.08x0.95mm_HandSolder
- J2: value Conn_01x08_Socket -> 01x08_Socket
- J3: value Conn_01x04_Socket -> 01x04_Socket
- S1, S2, S3, S4: footprint samacsys:TVGP01G73BB -> SamacSys_Parts:TVGP01G73BB
- moved SW1 12.4 mm to (146.6, 60.7)
- moved SW2 11.3 mm to (135.4, 60.7)
- moved J2 0.76 mm to (156.2, 145.3)
- moved JP1 0.51 mm to (153.9, 81.3)
Connections:
- S1 pad 1: +3V3 -> GND
- S2 pad 1: +3V3 -> GND
- S3 pad 1: +3V3 -> GND
- S4 pad 1: +3V3 -> GND
- U1 pad 37: unconnected-(U1-75/IOT38A/RGB_R3/HDMI_D2P-Pad37) -> /SW3
Routing:
- net /SW3: track 0.00 -> 88.1 mm
- net +3V3: track 166.9 -> 126.8 mm
- net Net-(SW1-B): track 87.0 -> 74.7 mm
- net Net-(SW2-B): track 91.8 -> 81.4 mm
- net GND: track 0.00 -> 2.20 mm, vias 0 -> 12
- net Net-(J2-Pin_8): track 4.62 -> 3.85 mm
- net Net-(J2-Pin_7): track 4.62 -> 3.85 mm
- net Net-(J2-Pin_6): track 4.62 -> 3.85 mm
- net Net-(J2-Pin_5): track 4.62 -> 3.85 mm
- net Net-(J2-Pin_4): track 4.62 -> 3.85 mm
- net Net-(J2-Pin_3): track 4.62 -> 3.85 mm
- net Net-(J2-Pin_2): track 4.62 -> 3.85 mm
- net Net-(J2-Pin_1): track 4.62 -> 3.85 mm
- net Net-(S4-NO_1): track 24.2 -> 23.6 mm
- net Net-(S2-NO_1): track 45.7 -> 46.2 mm
Other:
- board text added: "80"
- board text added: "81"
- board text added: "82"
- board text added: "83"
- board text added: "84"
- board text added: "85"
- board text added: "A2"
- board text added: "A3"
- board text added: "A4"
- board text added: "A5"
- board text added: "A6"
- board text added: "A7"

Commit message: 0916
Connections:
- U1 pad 18: unconnected-(U1-53/IOR15B/RGB_B4-Pad18) -> /HIN_T
- U1 pad 19: unconnected-(U1-54/IOR15A/RGB_B3-Pad19) -> /HIN_R
- U1 pad 20: unconnected-(U1-55/IOR14B/RGB_G7-Pad20) -> /HIN_S
Routing:
- net /HIN_T: track 0.00 -> 28.1 mm
- net /HIN_S: track 0.00 -> 18.8 mm
- net /HIN_R: track 0.00 -> 18.2 mm
- net GND: vias 12 -> 11

Commit message: 0916
Parts:
- renumbered J1 to CN1
Changed lines of the file:
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@@
     (property "ki_description" "Tactile Switch")
     (attr through_hole)
-    (fp_text reference "S1" (at 6.25 2.5) (layer "F.SilkS")
+    (fp_text reference "S1" (at 6.25 9.485) (layer "F.SilkS")
         (effects (font (size 1.27 1.27) (thickness 0.254)))
     )
@@
     (property "ki_description" "Tactile Switch")
     (attr through_hole)
-    (fp_text reference "S2" (at 6.25 2.5 180) (layer "F.SilkS")
+    (fp_text reference "S2" (at 6.25 -4.485 180) (layer "F.SilkS")
         (effects (font (size 1.27 1.27) (thickness 0.254)))
     )
@@
     (property "ki_keywords" "connector")
     (attr through_hole)
-    (fp_text reference "J1" (at 1.27 -2.77) (layer "F.SilkS")
+    (fp_text reference "CN1" (at 1.27 -2.77) (layer "F.SilkS")
         (effects (font (size 1 1) (thickness 0.15)))
     )
@@
     (property "ki_description" "Tactile Switch")
     (attr through_hole)
-    (fp_text reference "S3" (at 6.25 2.5) (layer "F.SilkS")
+    (fp_text reference "S3" (at 6.277 9.525) (layer "F.SilkS")
         (effects (font (size 1.27 1.27) (thickness 0.254)))
     )
@@
     (property "ki_description" "Tactile Switch")
     (attr through_hole)
-    (fp_text reference "S4" (at 6.25 2.5) (layer "F.SilkS")
+    (fp_text reference "S4" (at 6.25 9.485) (layer "F.SilkS")
         (effects (font (size 1.27 1.27) (thickness 0.254)))
     )
@@
     (effects (font (size 1 1) (thickness 0.15)) (justify left bottom))
   )
-  (gr_text "37" (at 187.452 135.382) (layer "F.SilkS")
+  (gr_text "37" (at 187.96 135.382) (layer "F.SilkS")
     (effects (font (size 0.7 0.7) (thickness 0.15)) (justify left bottom))
   )
@@
     (effects (font (size 1 1) (thickness 0.15)) (justify left bottom))
   )
-  (gr_text "37" (at 126.238 135.382) (layer "F.SilkS")
+  (gr_text "37" (at 127 135.382) (layer "F.SilkS")
     (effects (font (size 0.7 0.7) (thickness 0.15)) (justify left bottom))
   )

Commit message: 0917
Connections:
- J3 pad 1: Net-(J3-Pin_1) -> /_LIN_S
- J3 pad 2: Net-(J3-Pin_2) -> /_LIN_R
- J3 pad 3: Net-(J3-Pin_3) -> /_LIN_T
- U1 pad 1: Net-(J3-Pin_1) -> /_LIN_S
- U1 pad 2: Net-(J3-Pin_2) -> /_LIN_R
- U1 pad 3: Net-(J3-Pin_3) -> /_LIN_T
Routing:
- net /_LIN_S: track 0.00 -> 87.8 mm
- net /_LIN_R: track 0.00 -> 46.0 mm
- net /_LIN_T: track 0.00 -> 41.7 mm
- net Net-(J3-Pin_3): track 4.95 -> 0.00 mm
- net Net-(J3-Pin_2): track 4.95 -> 0.00 mm
- net Net-(J3-Pin_1): track 4.95 -> 0.00 mm
- net GND: vias 11 -> 13
Other:
- board text added: "36/#LIN_T"
- board text added: "37/#LIN_R"
- board text added: "38/#LIN_S"
- board text added: "Tang Nano 9K - InverterKit2"
