File: tangnano9k_brushless_driver.kicad_pcb (KiCad board)
At the start: 2 copper layers, 81.5 x 99.9 mm, 27 parts, among them CN1 Nucleo_F302R8, J2 01x08_Socket, J3 01x04_Socket, SW1 SW_SPDT, SW2 SW_SPDT, SW3 SW_SPDT, U1 Tang_Nano_9k_board, U2 MCP3008, U3 C-574SR-LF

Commit message: 0921
Parts:
- moved G*** 1.15 mm to (129.2, 75.8)
- renumbered SW1 to Reverse
Other:
- board text added: "0"
- board text added: "Motor"
- board text added: "|"
Changed lines of the file:
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@@
     (property "ki_keywords" "switch single-pole double-throw spdt ON-ON")
     (attr through_hole)
-    (fp_text reference "SW1" (at -2.794 -3.81) (layer "F.SilkS")
+    (fp_text reference "Reverse" (at 0 -3.683) (layer "F.SilkS")
         (effects (font (size 1 1) (thickness 0.15)))
     )
@@
     (property "ki_keywords" "switch single-pole double-throw spdt ON-ON")
     (attr through_hole)
-    (fp_text reference "SW2" (at -2.794 -3.81) (layer "F.SilkS")
+    (fp_text reference "SW2" (at -0.127 -3.683) (layer "F.SilkS")
         (effects (font (size 1 1) (thickness 0.15)))
     )
@@
     (property "ki_keywords" "switch single-pole double-throw spdt ON-ON")
     (attr through_hole)
-    (fp_text reference "SW3" (at -3.048 -3.81) (layer "F.SilkS")
+    (fp_text reference "SW3" (at -3.048 -3.81) (layer "F.SilkS") hide
         (effects (font (size 1 1) (thickness 0.15)))
     )
@@
   )
   (footprint "MyLibrary:kamo20" (layer "F.Cu")
-    (at 129.032 74.676)
+    (at 129.159 75.819)
     (attr board_only exclude_from_pos_files exclude_from_bom)
     (fp_text reference "G***" (at 0 0) (layer "F.SilkS") hide
@@
     (property "ki_keywords" "connector")
     (attr through_hole)
-    (fp_text reference "U3" (at -4.172 -1.016) (layer "F.SilkS")
+    (fp_text reference "U3" (at -3.029 0.254) (layer "F.SilkS")
         (effects (font (size 1 1) (thickness 0.15)))
     )
@@
     (effects (font (size 1 1) (thickness 0.15)) (justify left bottom))
   )
+  (gr_text "Motor" (at 121.666 57.531) (layer "F.SilkS")
+    (effects (font (size 1 1) (thickness 0.15)) (justify left bottom))
+  )
   (gr_text "[BP5293-50]" (at 142.24 111.125 90) (layer "F.SilkS")
     (effects (font (size 1 1) (thickness 0.15)) (justify left bottom))
@@
     (effects (font (size 1 1) (thickness 0.15)) (justify left bottom))
   )
+  (gr_text "0" (at 123.444 59.055) (layer "F.SilkS")
+    (effects (font (size 1 1) (thickness 0.15)) (justify left bottom))
+  )
   (gr_text "DIG1" (at 173.863 65.532 90) (layer "F.SilkS")
     (effects (font (size 1 1) (thickness 0.15)) (justify left bottom))
@@
     (effects (font (size 1 1) (thickness 0.15)) (justify left bottom))
   )
+  (gr_text "0" (at 134.874 59.055) (layer "F.SilkS")
+    (effects (font (size 1 1) (thickness 0.15)) (justify left bottom))
+  )
   (gr_text "A5" (at 139.192 90.678) (layer "F.SilkS")
     (effects (font (size 1 1) (thickness 0.15)) (justify left bottom))
@@
     (effects (font (size 1 1) (thickness 0.15)) (justify left bottom))
   )
+  (gr_text "0" (at 146.05 59.055) (layer "F.SilkS")
+    (effects (font (size 1 1) (thickness 0.15)) (justify left bottom))
+  )
   (gr_text "39" (at 189.484 140.843) (layer "F.SilkS")
     (effects (font (size 1 1) (thickness 0.15)) (justify left bottom))
@@
     (effects (font (size 1 1) (thickness 0.15)) (justify left bottom))
   )
+  (gr_text "|" (at 123.444 68.834) (layer "F.SilkS")
+    (effects (font (size 1 1) (thickness 0.15)) (justify left bottom))
+  )
   (gr_text "CLK" (at 150.876 88.138) (layer "F.SilkS")
     (effects (font (size 1 1) (thickness 0.15)) (justify left bottom))
@@
     (effects (font (size 1 1) (thickness 0.15)) (justify left bottom))
   )
+  (gr_text "|" (at 146.05 68.707) (layer "F.SilkS")
+    (effects (font (size 1 1) (thickness 0.15)) (justify left bottom))
+  )
   (gr_text "37/#LIN_R" (at 189.484 145.923) (layer "F.SilkS")
     (effects (font (size 1 1) (thickness 0.15)) (justify left bottom))
@@
     (effects (font (size 1 1) (thickness 0.15)) (justify left bottom))
   )
+  (gr_text "|" (at 134.874 68.707) (layer "F.SilkS")
+    (effects (font (size 1 1) (thickness 0.15)) (justify left bottom))
+  )
