File: tangnano9k_brushless_driver.kicad_sch (KiCad schematic)
At the start: 2 parts, among them J1 Nucleo_F302R8, U1 Tang_Nano_9k_board

Commit message: 0905
Parts:
- added PS1: BP5293-50, TO254P570X1700X1780-3P, symbol samacsys:BP5293-50
Connections:
- net DIRECTION: now also U1.21 (56/IOR14A/RGB_G6)
- net D_IN: now also U1.22 (57/IOR13A/RGB_G5)
- net HIN_R: now also U1.24 (69/IOT42A/RGB_G3/HDMI_CKP); no longer U1.22 (57/IOR13A/RGB_G5)
- net HIN_S: now also U1.23 (68/IOT42B/RGB_G4/HDMI_CKN); no longer U1.20 (55/IOR14B/RGB_G7)
- net VIN12: now also PS1.1 (VIN)
- net _LIN_R: now also U1.19 (54/IOR15A/RGB_B3); no longer U1.21 (56/IOR14A/RGB_G6)
- net _LIN_S: now also U1.17 (51/IOR17B/RGB_B5); no longer U1.19 (54/IOR15A/RGB_B3)
- net _LIN_T: now also U1.20 (55/IOR14B/RGB_G7); no longer U1.17 (51/IOR17B/RGB_B5)
- net 3.3V: now reaches U1.25 (3V3)
- net 3.3V: now also J1.16 (Pin_16)
- net GND: now reaches U1.26 (GND)
- net GND: now also J1.19 (Pin_19), J1.20 (Pin_20), J1.22 (Pin_22), J1.47, J1.58, J1.70, J1.8 (Pin_8), PS1.2 (GND)
- net 5V: now reaches U1.31 (5V)
- net 5V: now also J1.18 (Pin_18), PS1.3 (VOUT)
- net C7-28: now reaches J1.28 (Pin_28)
- net C7-30: now reaches J1.30 (Pin_30)
- net C7-36: now reaches J1.36 (Pin_36)
- net U: now reaches J1.37 (Pin_37)
- net C7-38: now reaches J1.38 (Pin_38)
- net C10-01: now reaches J1.39
- net C10-11: now reaches J1.49
- net V: now reaches J1.56
- net C10-28: now reaches J1.66
- net C10-34: now reaches J1.72
- no-connect marks 0 -> 43

Commit message: 0905
Parts:
- added C1: C, Capacitor_THT:C_Axial_L3.8mm_D2.6mm_P7.50mm_Horizontal, symbol Device:C
- added J2: Conn_01x08_Socket, Connector_PinSocket_2.54mm:PinSocket_1x08_P2.54mm_Vertical, symbol Connector:Conn_01x08_Socket
- added U2: MCP3008, Package_DIP:DIP-16_W7.62mm, symbol Analog_ADC:MCP3008
- J1: footprint (none) -> Library:Nucleo
- PS1: footprint TO254P570X1700X1780-3P -> samacsys:TO254P570X1700X1780-3P
- U1: footprint Custom Library:Tang Nano 9K -> Library:Tang Nano 9K
Connections:
- net ACCEL: now also U2.7 (CH6)
- net A_IN: now also U2.6 (CH5)
- net C10-11: now also U2.8 (CH7)
- net C10-28: now also U2.4 (CH3)
- net C10-34: now also U2.5 (CH4)
- net C7-28: now also U2.1 (CH0)
- net C7-36: now also U2.2 (CH1)
- net C7-38: now also U2.3 (CH2)
- net GND: now also C1.2, U2.14 (AGND), U2.9 (DGND)
- net at U1.15 (41/IOB41A/RGB_B7): now also U2.10 (~{CS}/SHDN)
- net at U1.16 (42IOB41B/RGB_B6): now also U2.11 (Din)
- net at U1.27 (32/IOB15B/RGB_TOUCH_XR): now also U2.13 (CLK)
- net at U1.28 (31/IOB15A/RGB_TOUCH_YD): now also U2.12 (Dout)
- net at U1.40 (79/IOT12B): now also J2.8 (Pin_8)
- net at U1.41 (80/IOT12A): now also J2.7 (Pin_7)
- net at U1.42 (81/IOT11B): now also J2.6 (Pin_6)
- net at U1.43 (82/IOT11A): now also J2.5 (Pin_5)
- net at U1.44 (83/IOT10B): now also J2.4 (Pin_4)
- net at U1.45 (84/IOT10A): now also J2.3 (Pin_3)
- net at U1.46 (85/IOT8B): now also J2.2 (Pin_2)
- net at U1.47 (86/IOT8A/RGB_BL): now also J2.1 (Pin_1)
- net 3.3V renamed +3.3V
- net +3.3V: now also C1.1, U2.15 (Vref), U2.16 (Vdd)
Other:
- moved on the sheet: J1, PS1, U1

Commit message: 0906
Connections:
- net DIRECTION: now also U1.24 (69/IOT42A/RGB_G3/HDMI_CKP); no longer U1.21 (56/IOR14A/RGB_G6)
- net D_IN: now also U1.23 (68/IOT42B/RGB_G4/HDMI_CKN); no longer U1.22 (57/IOR13A/RGB_G5)
- net HIN_R: no longer U1.24 (69/IOT42A/RGB_G3/HDMI_CKP)
- net HIN_S: no longer U1.23 (68/IOT42B/RGB_G4/HDMI_CKN)
- net HIN_T: no longer U1.18 (53/IOR15B/RGB_B4)
- net H_V: now also U1.12 (34/IOB23B/RGB_VS); no longer U1.9 (29/IOB13A)
- net H_W: now also U1.13 (40/IOB33B/RGB_HS); no longer U1.8 (28/IOB11B)
- net _LIN_R: no longer U1.19 (54/IOR15A/RGB_B3)
- net _LIN_S: no longer U1.17 (51/IOR17B/RGB_B5)
- net _LIN_T: no longer U1.20 (55/IOR14B/RGB_G7)
Changed lines of the file:
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@@
-    (stroke (width 0) (type default))
-  )
-  (wire (pts (xy 199.39 111.76) (xy 199.39 33.02))
     (stroke (width 0) (type default))
   )
@@
     (stroke (width 0) (type default))
   )
-  (wire (pts (xy 86.36 106.045) (xy 86.36 52.07))
+  (wire (pts (xy 86.36 36.83) (xy 86.36 106.045))
     (stroke (width 0) (type default))
   )
@@
     (stroke (width 0) (type default))
   )
-  (wire (pts (xy 85.09 49.53) (xy 101.6 49.53))
-    (stroke (width 0) (type default))
-  )
   (wire (pts (xy 49.53 73.025) (xy 49.53 84.455))
     (stroke (width 0) (type default))
@@
     (stroke (width 0) (type default))
   )
+  (wire (pts (xy 199.39 111.76) (xy 199.39 43.18))
+    (stroke (width 0) (type default))
+  )
   (wire (pts (xy 142.875 123.825) (xy 142.875 109.855))
     (stroke (width 0) (type default))
@@
     (stroke (width 0) (type default))
   )
+  (wire (pts (xy 166.37 40.64) (xy 198.12 40.64))
+    (stroke (width 0) (type default))
+  )
   (wire (pts (xy 166.37 88.9) (xy 167.64 88.9))
     (stroke (width 0) (type default))
@@
     (stroke (width 0) (type default))
   )
-  (wire (pts (xy 199.39 33.02) (xy 166.37 33.02))
-    (stroke (width 0) (type default))
-  )
   (wire (pts (xy 110.49 151.765) (xy 128.905 151.765))
     (stroke (width 0) (type default))
   )
-  (wire (pts (xy 195.58 107.95) (xy 195.58 40.64))
-    (stroke (width 0) (type default))
-  )
   (wire (pts (xy 141.605 144.145) (xy 141.605 107.95))
     (stroke (width 0) (type default))
   )
-  (wire (pts (xy 197.485 109.855) (xy 197.485 35.56))
+  (wire (pts (xy 198.12 109.855) (xy 198.12 40.64))
     (stroke (width 0) (type default))
   )
@@
     (stroke (width 0) (type default))
   )
-  (wire (pts (xy 166.37 30.48) (xy 201.295 30.48))
-    (stroke (width 0) (type default))
-  )
   (wire (pts (xy 171.45 141.605) (xy 177.165 141.605))
     (stroke (width 0) (type default))
@@
     (stroke (width 0) (type default))
   )
+  (wire (pts (xy 85.09 39.37) (xy 101.6 39.37))
+    (stroke (width 0) (type default))
+  )
   (wire (pts (xy 158.75 156.845) (xy 137.795 156.845))
     (stroke (width 0) (type default))
@@
     (stroke (width 0) (type default))
   )
-  (wire (pts (xy 142.875 109.855) (xy 197.485 109.855))
+  (wire (pts (xy 142.875 109.855) (xy 198.12 109.855))
     (stroke (width 0) (type default))
   )
@@
     (stroke (width 0) (type default))
   )
-  (wire (pts (xy 203.2 27.94) (xy 166.37 27.94))
-    (stroke (width 0) (type default))
-  )
   (wire (pts (xy 215.265 30.48) (xy 224.155 30.48))
     (stroke (width 0) (type default))
   )
-  (wire (pts (xy 195.58 40.64) (xy 166.37 40.64))
-    (stroke (width 0) (type default))
-  )
   (wire (pts (xy 141.605 107.95) (xy 195.58 107.95))
     (stroke (width 0) (type default))
@@
     (stroke (width 0) (type default))
   )
-  (wire (pts (xy 205.105 25.4) (xy 166.37 25.4))
-    (stroke (width 0) (type default))
-  )
   (wire (pts (xy 158.75 159.385) (xy 138.43 159.385))
     (stroke (width 0) (type default))
@@
     (stroke (width 0) (type default))
   )
+  (wire (pts (xy 166.37 43.18) (xy 199.39 43.18))
+    (stroke (width 0) (type default))
+  )
   (wire (pts (xy 97.79 139.065) (xy 83.82 139.065))
     (stroke (width 0) (type default))
   )
-  (wire (pts (xy 86.36 52.07) (xy 101.6 52.07))
+  (wire (pts (xy 86.36 36.83) (xy 101.6 36.83))
     (stroke (width 0) (type default))
   )
@@
     (stroke (width 0) (type default))
   )
-  (wire (pts (xy 85.09 107.315) (xy 85.09 49.53))
+  (wire (pts (xy 85.09 39.37) (xy 85.09 107.315))
     (stroke (width 0) (type default))
   )
@@
     (stroke (width 0) (type default))
   )
-  (wire (pts (xy 207.01 22.86) (xy 166.37 22.86))
-    (stroke (width 0) (type default))
-  )
   (wire (pts (xy 98.425 91.44) (xy 101.6 91.44))
     (stroke (width 0) (type default))
@@
     (stroke (width 0) (type default))
   )
-  (wire (pts (xy 193.675 43.18) (xy 166.37 43.18))
-    (stroke (width 0) (type default))
-  )
-  (wire (pts (xy 197.485 35.56) (xy 166.37 35.56))
-    (stroke (width 0) (type default))
-  )
-  (wire (pts (xy 193.675 106.045) (xy 193.675 43.18))
-    (stroke (width 0) (type default))
-  )

Commit message: 0907
Parts:
- added JP1: SolderJumper_2_Open, Jumper:SolderJumper-2_P1.3mm_Open_TrianglePad1.0x1.5mm, symbol Jumper:SolderJumper_2_Open
- added R1, R2: R, Resistor_SMD:R_0603_1608Metric_Pad0.98x0.95mm_HandSolder, symbol Device:R
- C1: footprint Capacitor_THT:C_Axial_L3.8mm_D2.6mm_P7.50mm_Horizontal -> Capacitor_SMD:C_0603_1608Metric_Pad1.08x0.95mm_HandSolder
Connections:
- net +3.3V: now also JP1.2 (B), R1.1; no longer C1.1, U2.15 (Vref)
- net ACCEL: now also U2.5 (CH4); no longer U2.7 (CH6)
- net A_IN: now also U2.7 (CH6); no longer U2.6 (CH5)
- net C10-11: now also U2.1 (CH0); no longer U2.8 (CH7)
- net C10-28: now also U2.2 (CH1); no longer U2.4 (CH3)
- net C10-34: now also U2.3 (CH2); no longer U2.5 (CH4)
- net C7-28: now also U2.8 (CH7); no longer U2.1 (CH0)
- net C7-36: now also U2.6 (CH5); no longer U2.2 (CH1)
- net C7-38: now also U2.4 (CH3); no longer U2.3 (CH2)
- net GND: now also R2.2
- net H_U: now also U1.11 (33/IOB23A/RGB_DE); no longer U1.10 (30/IOB13B)
- new net: C1.1, JP1.1 (A), R1.2, R2.1, U2.15 (Vref)
Changed lines of the file:
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@@
   (junction (at 35.56 60.325) (diameter 0) (color 0 0 0 0)
+  )
+  (junction (at 24.765 60.325) (diameter 0) (color 0 0 0 0)
+  )
+  (junction (at 35.56 52.705) (diameter 0) (color 0 0 0 0)
+  )
+  (junction (at 30.48 52.705) (diameter 0) (color 0 0 0 0)
+  )
+  (junction (at 35.56 67.945) (diameter 0) (color 0 0 0 0)
+  )
+  (junction (at 30.48 60.325) (diameter 0) (color 0 0 0 0)
   )
   (junction (at 112.395 141.605) (diameter 0) (color 0 0 0 0)
@@
     (stroke (width 0) (type default))
   )
+  (wire (pts (xy 24.765 60.325) (xy 30.48 60.325))
+    (stroke (width 0) (type default))
+  )
   (wire (pts (xy 84.455 164.465) (xy 97.79 164.465))
     (stroke (width 0) (type default))
   )
+  (wire (pts (xy 83.82 41.91) (xy 83.82 139.065))
+    (stroke (width 0) (type default))
+  )
   (wire (pts (xy 201.295 146.685) (xy 201.295 30.48))
     (stroke (width 0) (type default))
@@
     (stroke (width 0) (type default))
   )
+  (wire (pts (xy 30.48 52.705) (xy 35.56 52.705))
+    (stroke (width 0) (type default))
+  )
   (wire (pts (xy 98.425 76.2) (xy 101.6 76.2))
     (stroke (width 0) (type default))
@@
     (stroke (width 0) (type default))
   )
-  (wire (pts (xy 83.82 46.99) (xy 101.6 46.99))
-    (stroke (width 0) (type default))
-  )
   (wire (pts (xy 110.49 159.385) (xy 136.525 159.385))
     (stroke (width 0) (type default))
@@
     (stroke (width 0) (type default))
   )
+  (wire (pts (xy 30.48 60.325) (xy 35.56 60.325))
+    (stroke (width 0) (type default))
+  )
   (wire (pts (xy 207.01 172.085) (xy 207.01 22.86))
     (stroke (width 0) (type default))
@@
     (stroke (width 0) (type default))
   )
-  (wire (pts (xy 83.82 139.065) (xy 83.82 46.99))
-    (stroke (width 0) (type default))
-  )
   (wire (pts (xy 171.45 146.685) (xy 201.295 146.685))
     (stroke (width 0) (type default))
@@
     (stroke (width 0) (type default))
   )
+  (wire (pts (xy 83.82 41.91) (xy 101.6 41.91))
+    (stroke (width 0) (type default))
+  )
+  (wire (pts (xy 24.765 52.705) (xy 30.48 52.705))
+    (stroke (width 0) (type default))
+  )
   (wire (pts (xy 57.15 31.75) (xy 101.6 31.75))
     (stroke (width 0) (type default))
@@
     (stroke (width 0) (type default))
   )
+  (wire (pts (xy 24.765 67.945) (xy 35.56 67.945))
+    (stroke (width 0) (type default))
+  )
   (wire (pts (xy 98.425 81.28) (xy 101.6 81.28))
     (stroke (width 0) (type default))
@@
     (effects (font (size 1.27 1.27)) (justify left bottom))
   )
-  (label "C7-36" (at 46.99 82.55 90) (fields_autoplaced)
-    (effects (font (size 1.27 1.27)) (justify left bottom))
-  )
-  (label "C10-28" (at 52.07 82.55 90) (fields_autoplaced)
+  (label "C10-11" (at 44.45 82.55 90) (fields_autoplaced)
     (effects (font (size 1.27 1.27)) (justify left bottom))
   )
@@
     (effects (font (size 1.27 1.27)) (justify left bottom))
   )
+  (label "A_IN" (at 59.69 80.645 90) (fields_autoplaced)
+    (effects (font (size 1.27 1.27)) (justify left bottom))
+  )
   (label "_LIN_R" (at 173.99 149.225 0) (fields_autoplaced)
     (effects (font (size 1.27 1.27)) (justify left bottom))
@@
     (effects (font (size 1.27 1.27)) (justify left bottom))
   )
+  (label "ACCEL" (at 54.61 81.28 90) (fields_autoplaced)
+    (effects (font (size 1.27 1.27)) (justify left bottom))
+  )
   (label "ACCEL" (at 90.17 161.925 0) (fields_autoplaced)
     (effects (font (size 1.27 1.27)) (justify left bottom))
   )
-  (label "C10-34" (at 54.61 82.55 90) (fields_autoplaced)
+  (label "C10-34" (at 49.53 81.28 90) (fields_autoplaced)
     (effects (font (size 1.27 1.27)) (justify left bottom))
   )
@@
     (effects (font (size 1.27 1.27)) (justify left bottom))
   )
-  (label "C7-38" (at 49.53 82.55 90) (fields_autoplaced)
-    (effects (font (size 1.27 1.27)) (justify left bottom))
-  )
   (label "U" (at 91.44 164.465 0) (fields_autoplaced)
     (effects (font (size 1.27 1.27)) (justify left bottom))
   )
-  (label "ACCEL" (at 59.69 81.915 90) (fields_autoplaced)
-    (effects (font (size 1.27 1.27)) (justify left bottom))
-  )
   (label "C10-34" (at 171.45 159.385 0) (fields_autoplaced)
     (effects (font (size 1.27 1.27)) (justify left bottom))
@@
     (effects (font (size 1.27 1.27)) (justify left bottom))
   )
-  (label "A_IN" (at 57.15 81.915 90) (fields_autoplaced)
-    (effects (font (size 1.27 1.27)) (justify left bottom))
-  )
   (label "HIN_R" (at 140.335 146.685 0) (fields_autoplaced)
     (effects (font (size 1.27 1.27)) (justify left bottom))
@@
     (effects (font (size 1.27 1.27)) (justify left bottom))
   )
-  (label "C7-28" (at 44.45 82.55 90) (fields_autoplaced)
-    (effects (font (size 1.27 1.27)) (justify left bottom))
-  )
   (label "C10-28" (at 173.99 151.765 0) (fields_autoplaced)
     (effects (font (size 1.27 1.27)) (justify left bottom))
   )
+  (label "C7-38" (at 52.07 81.28 90) (fields_autoplaced)
+    (effects (font (size 1.27 1.27)) (justify left bottom))
+  )
   (label "H_W" (at 154.305 149.225 0) (fields_autoplaced)
     (effects (font (size 1.27 1.27)) (justify left bottom))
   )
+  (label "C7-28" (at 62.23 81.28 90) (fields_autoplaced)
+    (effects (font (size 1.27 1.27)) (justify left bottom))
+  )
   (label "HIN_S" (at 152.4 144.145 0) (fields_autoplaced)
     (effects (font (size 1.27 1.27)) (justify left bottom))
@@
     (effects (font (size 1.27 1.27)) (justify left bottom))
   )
+  (label "C10-28" (at 46.99 81.915 90) (fields_autoplaced)
+    (effects (font (size 1.27 1.27)) (justify left bottom))
+  )
   (label "DIRECTION" (at 148.59 121.285 0) (fields_autoplaced)
     (effects (font (size 1.27 1.27)) (justify left bottom))
@@
     (effects (font (size 1.27 1.27)) (justify left bottom))
   )
-  (label "C10-11" (at 62.23 81.915 90) (fields_autoplaced)
+  (label "C7-36" (at 57.15 81.28 90) (fields_autoplaced)
     (effects (font (size 1.27 1.27)) (justify left bottom))
   )
@@
     )
   )
+  (symbol (lib_id "Device:R") (at 24.765 64.135 0) (unit 1)
+    (in_bom yes) (on_board yes) (dnp no) (fields_autoplaced)
+    (property "Reference" "R2" (at 26.67 63.5 0)
+      (effects (font (size 1.27 1.27)) (justify left))
+    )
+    (property "Value" "R" (at 26.67 66.04 0)
+      (effects (font (size 1.27 1.27)) (justify left))
+    )
+    (property "Footprint" "Resistor_SMD:R_0603_1608Metric_Pad0.98x0.95mm_HandSolder" (at 22.987 64.135 90)
+      (effects (font (size 1.27 1.27)) hide)
+    )
+    (property "Datasheet" "~" (at 24.765 64.135 0)
+      (effects (font (size 1.27 1.27)) hide)
+    )
+    (pin "1")
+    (pin "2")
+    (instances
+      (project "tangnano9k_brushless_driver"
+        (path "/8aff725f-ee01-408d-a4eb-7fb705fecf00"
+          (reference "R2") (unit 1)
+        )
+      )
+    )
+  )
   (symbol (lib_id "power:+3.3V") (at 174.625 91.44 0) (unit 1)
     (in_bom yes) (on_board yes) (dnp no) (fields_autoplaced)
@@
       (effects (font (size 1.27 1.27)) (justify left))
     )
-    (property "Footprint" "Capacitor_THT:C_Axial_L3.8mm_D2.6mm_P7.50mm_Horizontal" (at 36.5252 67.945 0)
+    (property "Footprint" "Capacitor_SMD:C_0603_1608Metric_Pad1.08x0.95mm_HandSolder" (at 36.5252 67.945 0)
       (effects (font (size 1.27 1.27)) hide)
     )
@@
         (path "/8aff725f-ee01-408d-a4eb-7fb705fecf00"
           (reference "C1") (unit 1)
+        )
+      )
+    )
+  )
+  (symbol (lib_id "Jumper:SolderJumper_2_Open") (at 30.48 56.515 90) (unit 1)
+    (in_bom yes) (on_board yes) (dnp no) (fields_autoplaced)
+    (property "Reference" "JP1" (at 33.02 55.88 90)
+      (effects (font (size 1.27 1.27)) (justify right))
+    )
+    (property "Value" "SolderJumper_2_Open" (at 33.02 58.42 90)
+      (effects (font (size 1.27 1.27)) (justify right))
+    )
+    (property "Footprint" "Jumper:SolderJumper-2_P1.3mm_Open_TrianglePad1.0x1.5mm" (at 30.48 56.515 0)
+      (effects (font (size 1.27 1.27)) hide)
+    )
+    (property "Datasheet" "~" (at 30.48 56.515 0)
+      (effects (font (size 1.27 1.27)) hide)
+    )
+    (pin "1")
+    (pin "2")
+    (instances
+      (project "tangnano9k_brushless_driver"
+        (path "/8aff725f-ee01-408d-a4eb-7fb705fecf00"
+          (reference "JP1") (unit 1)
         )
       )
@@
     )
   )
-  (symbol (lib_id "power:+3.3V") (at 35.56 60.325 0) (unit 1)
-    (in_bom yes) (on_board yes) (dnp no) (fields_autoplaced)
-    (property "Reference" "#PWR012" (at 35.56 64.135 0)
-      (effects (font (size 1.27 1.27)) hide)
-    )
-    (property "Value" "+3.3V" (at 35.56 55.245 0)
-      (effects (font (size 1.27 1.27)))
-    )
-    (property "Footprint" "" (at 35.56 60.325 0)
-      (effects (font (size 1.27 1.27)) hide)
-    )
-    (property "Datasheet" "" (at 35.56 60.325 0)
-      (effects (font (size 1.27 1.27)) hide)
-    )
-    (pin "1")
-    (instances
-      (project "tangnano9k_brushless_driver"
-        (path "/8aff725f-ee01-408d-a4eb-7fb705fecf00"
-          (reference "#PWR012") (unit 1)
-        )
-      )
-    )
-  )
   (symbol (lib_id "power:GND") (at 211.455 33.02 0) (unit 1)
     (in_bom yes) (on_board yes) (dnp no) (fields_autoplaced)
@@
         )
       )
+    )
+  )
+  (symbol (lib_id "Device:R") (at 24.765 56.515 0) (unit 1)
+    (in_bom yes) (on_board yes) (dnp no) (fields_autoplaced)
+    (property "Reference" "R1" (at 26.67 55.88 0)
+      (effects (font (size 1.27 1.27)) (justify left))
+    )
+    (property "Value" "R" (at 26.67 58.42 0)
+      (effects (font (size 1.27 1.27)) (justify left))
+    )
+    (property "Footprint" "Resistor_SMD:R_0603_1608Metric_Pad0.98x0.95mm_HandSolder" (at 22.987 56.515 90)
+      (effects (font (size 1.27 1.27)) hide)
+    )
+    (property "Datasheet" "~" (at 24.765 56.515 0)
+      (effects (font (size 1.27 1.27)) hide)
+    )
+    (pin "1")
+    (pin "2")
+    (instances
+      (project "tangnano9k_brushless_driver"
+        (path "/8aff725f-ee01-408d-a4eb-7fb705fecf00"
+          (reference "R1") (unit 1)
+        )
+      )

Commit message: 0908
Parts:
- added J3: Conn_01x04_Socket, Connector_PinSocket_2.54mm:PinSocket_1x04_P2.54mm_Vertical, symbol Connector:Conn_01x04_Socket
- added R10, R3, R4, R5, R6, R7, R8, R9: R, Resistor_SMD:R_0603_1608Metric_Pad0.98x0.95mm_HandSolder, symbol Device:R
- added S1, S2, S3, S4: TVGP01-G73BB, TVGP01G73BB, symbol samacsys:TVGP01-G73BB
- added SW1, SW2: SW_SPDT, Connector_PinHeader_2.54mm:PinHeader_1x03_P2.54mm_Vertical, symbol Switch:SW_SPDT
- added U3: C-574SR-LF, Library:C-574SR-LF, symbol Library:C-574SR-LF
- C1: footprint Capacitor_SMD:C_0603_1608Metric_Pad1.08x0.95mm_HandSolder -> Connector:FanPinHeader_1x03_P2.54mm_Vertical
Connections:
- net GND: now also SW1.3 (C), SW2.3 (C)
- net H_U: now also U1.48 (63/IOR5A/RGB_TOUCH_XL); no longer U1.11 (33/IOB23A/RGB_DE)
- net H_V: now also U1.15 (41/IOB41A/RGB_B7); no longer U1.12 (34/IOB23B/RGB_VS)
- net H_W: now also U1.16 (42IOB41B/RGB_B6); no longer U1.13 (40/IOB33B/RGB_HS)
- net at U1.1 (38/IOB31B/TF_CS): now also J3.1 (Pin_1)
- net DIG1: now reaches U1.10 (30/IOB13B)
- net DIG1: now also U3.6 (Cathode_DIG4)
- net at U1.14 (35/IOB29A/RGB_CK): now also R10.2
- net CS/SHDN: now reaches U2.10 (~{CS}/SHDN)
- net CS/SHDN: now also U1.30 (48/IOR24B/SPILCD_CS); no longer U1.15 (41/IOB41A/RGB_B7)
- net Din: now reaches U2.11 (Din)
- net Din: now also U1.29 (49/IOR24A/SPILCD_RS); no longer U1.16 (42IOB41B/RGB_B6)
- net at U1.2 (37/IO31A/TF_MOSI): now also J3.2 (Pin_2)
- net Anode_A: now reaches U1.21 (56/IOR14A/RGB_G6)
- net Anode_A: now also R9.2
- net DIG4: now reaches U1.22 (57/IOR13A/RGB_G5)
- net DIG4: now also U3.12 (Cathode_DIG1)
- net at U1.3 (36/IOB29B/TF_SCK): now also J3.3 (Pin_3)
- net at U1.32 (70/IOT41B/RGB_G2/HDMI_C0N): now also S4.3 (NO_1)
- net at U1.33 (71/IOT41A/RGB_R7/HDMI_D0P): now also S3.3 (NO_1)
- net at U1.34 (72/IOT39B/RGB_R6/HDMI_D1N): now also S2.3 (NO_1)
- net at U1.35 (73/IOT39A/RGB_R5/HDMI_D1P): now also S1.3 (NO_1)
- net at U1.38 (76/IOT37B/SPILCD_CK): now also SW2.2 (B)
- net at U1.39 (77/IOT37A/SPILCD_MO): now also SW1.2 (B)
- net at U1.4 (39/IOB33A/TF_MISO): now also J3.4 (Pin_4)
- net at U1.5 (25/IOB8A): now also R3.2
- net at U1.6 (26/IOB8B): now also R4.2
- net at U1.7 (27/IOB11A): now also R5.2
- net at U1.8 (28/IOB11B): now also R6.2
- net at U1.9 (29/IOB13A): now also R7.2
- net +3.3V renamed +3V3
- net +3V3: now also S1.1 (COM_1), S2.1 (COM_1), S3.1 (COM_1), S4.1 (COM_1), SW1.1 (A), SW2.1 (A)
- new net: R8.2, U1.11 (33/IOB23A/RGB_DE)
- new net: R7.1, U3.5 (Anode_G)
- new net: R6.1, U3.4 (Anode_C)
- new net: R3.1, U3.1 (Anode_E)
- new net: R10.1, U3.10 (Anode_F)
- new net: R9.1, U3.11 (Anode_A)
- new net: R4.1, U3.2 (Anode_D)
- new net: R5.1, U3.3 (Anode_DP)
- new net: R8.1, U3.7 (Anode_B)
- new net DIG2: U1.13 (40/IOB33B/RGB_HS), U3.9 (Cathode_DIG2)
- new net DIG3: U1.12 (34/IOB23B/RGB_VS), U3.8 (Cathode_DIG3)
- no-connect marks 43 -> 51

Commit message: 0909
Parts:
- added SW3: SW_SPDT, Connector_PinHeader_2.54mm:PinHeader_1x03_P2.54mm_Vertical, symbol Switch:SW_SPDT
- C1: footprint Connector:FanPinHeader_1x03_P2.54mm_Vertical -> Capacitor_SMD:C_0603_1608Metric_Pad1.08x0.95mm_HandSolder
- J2: value Conn_01x08_Socket -> 01x08_Socket
- J3: value Conn_01x04_Socket -> 01x04_Socket
- S1, S2, S3, S4: footprint TVGP01G73BB -> SamacSys_Parts:TVGP01G73BB
Connections:
- net +3V3: now also SW3.1 (A); no longer S1.1 (COM_1), S2.1 (COM_1), S3.1 (COM_1), S4.1 (COM_1)
- net GND: now also S1.1 (COM_1), S2.1 (COM_1), S3.1 (COM_1), S4.1 (COM_1), SW3.3 (C)
- net SW3: now reaches U1.37 (75/IOT38A/RGB_R3/HDMI_D2P)
- net SW3: now also SW3.2 (B)
Other:
- moved on the sheet: R9, U3

Commit message: 0916
Connections:
- net HIN_R: now also U1.19 (54/IOR15A/RGB_B3)
- net HIN_S: now also U1.20 (55/IOR14B/RGB_G7)
- net HIN_T: now also U1.18 (53/IOR15B/RGB_B4)
Changed lines of the file:
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@@
+    (effects (font (size 1.27 1.27)) (justify left bottom))
+  )
+  (label "HIN_T" (at 166.37 25.4 0) (fields_autoplaced)
     (effects (font (size 1.27 1.27)) (justify left bottom))
   )
@@
     (effects (font (size 1.27 1.27)) (justify left bottom))
   )
+  (label "HIN_R" (at 166.37 27.94 0) (fields_autoplaced)
+    (effects (font (size 1.27 1.27)) (justify left bottom))
+  )
   (label "C7-30" (at 112.395 154.305 0) (fields_autoplaced)
     (effects (font (size 1.27 1.27)) (justify left bottom))
@@
     (effects (font (size 1.27 1.27)) (justify left bottom))
   )
+  (label "HIN_S" (at 166.37 30.48 0) (fields_autoplaced)
+    (effects (font (size 1.27 1.27)) (justify left bottom))
+  )
