File: tangnano9k_brushless_driver.kicad_sch (KiCad schematic)
At the start: 26 parts, among them J1 Nucleo_F302R8, J2 01x08_Socket, J3 01x04_Socket, SW1 SW_SPDT, SW2 SW_SPDT, SW3 SW_SPDT, U1 Tang_Nano_9k_board, U2 MCP3008, U3 C-574SR-LF

Commit message: 0917
Connections:
- net _LIN_R: now also J3.2 (Pin_2), U1.2 (37/IO31A/TF_MOSI)
- net _LIN_S: now also J3.1 (Pin_1), U1.1 (38/IOB31B/TF_CS)
- net _LIN_T: now also J3.3 (Pin_3), U1.3 (36/IOB29B/TF_SCK)
Changed lines of the file:
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@@
+    (effects (font (size 1.27 1.27)) (justify left bottom))
+  )
+  (label "_LIN_R" (at 98.425 69.85 0) (fields_autoplaced)
     (effects (font (size 1.27 1.27)) (justify left bottom))
   )
@@
     (effects (font (size 1.27 1.27)) (justify left bottom))
   )
+  (label "_LIN_S" (at 98.425 72.39 0) (fields_autoplaced)
+    (effects (font (size 1.27 1.27)) (justify left bottom))
+  )
   (label "C7-28" (at 62.23 81.28 90) (fields_autoplaced)
     (effects (font (size 1.27 1.27)) (justify left bottom))
@@
     (effects (font (size 1.27 1.27)) (justify left bottom))
   )
+  (label "_LIN_T" (at 98.425 67.31 0) (fields_autoplaced)
+    (effects (font (size 1.27 1.27)) (justify left bottom))
+  )
